Commit message: Add files via upload

File: turtlebot3_manipulation_description/urdf/turtlebot3_manipulation_robot.urdf.xacro (robot description, xacro)
@@ -2,10 +2,10 @@
 <robot name="turtlebot3_manipulation" xmlns:xacro="http://ros.org/wiki/xacro">
   <!-- Include TurtleBot3 Waffle URDF -->
-  <xacro:include filename="$(find turtlebot3_description)/urdf/turtlebot3_waffle_pi_for_open_manipulator.urdf.xacro"/>
+  <xacro:include filename="$(find turtlebot3_description)/urdf/turtlebot3_mecanum_with_open_manipulator.urdf.xacro"/>
   <!-- Include OpenMANIPULATOR URDF -->
   <xacro:include filename="$(find turtlebot3_manipulation_description)/urdf/open_manipulator_x.urdf.xacro"/>
   <!-- Base fixed joint -->
   <joint name="base_fixed" type="fixed">
-    <origin xyz="-0.092 0.0 0.091" rpy="0 0 0"/>
+    <origin xyz="-0.03 0.0 0.091" rpy="0 0 0"/>
     <parent link="base_link"/>
     <child link="link1"/>
